File: Hardwares/Aju_ver001/Aju_ver001.kicad_pcb (KiCad board)
At the start: 2 copper layers, 23 x 16 mm, 20 parts, among them CON1 53261-0271, CON2 FTM-103-02-F-DV, U1 RP110L251D-TR, U2 RP110L301D-TR, U3 ATtiny2313A-MU, U4 DRV8837, U5 DRV8837

Commit message: first commit
Connections:
- U1 pad 3: (no net) -> +BATT
- U2 pad 3: (no net) -> +BATT
Routing:
- net +BATT: track 47.7 -> 50.1 mm
